File: eagle/altera digital explorer.brd (EAGLE design)
At the start: 127 x 101.6 mm, 87 parts, among them IC1 EPM240T100C4, IC2 PIC18F14K50SO, IC3 MCP1703T-3302E/MB, J1 CON_HEADER_1X05-PTH, J8 MICRO-USB-5P-ZX62D-B-5P8-MILL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, Q1 12.00 MHz, SW1 SS-12E10, SW2 SS-12E10, SW3 SS-12E10, SW4 SS-12E10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

Commit message: PCB update: fix incorrect routing of JTAG programming outputs, change lighthouse to be CPLD controlled, add pushbuttons in addition to switch
Parts:
- added S1, S2, S3, S4, S5: (no value), SparkFun:TACTILE-PTH
- moved R9 25.3 mm to (40.3, 34.3)
- moved R8 22.3 mm to (40.3, 36.8)
- moved R6 21.2 mm to (40.3, 42.0)
- moved R7 20.7 mm to (40.3, 39.4)
- moved SW1 1.91 mm to (10.2, 49.5)
- moved SW2 1.27 mm to (10.2, 40.6)
- moved SW3 0.64 mm to (10.2, 31.8)
- moved SW5 0.63 mm to (10.2, 14.0)
Connections:
- removed net N$20: R20.1, SW4.RIGHT
- removed net N$21: R21.1, SW3.RIGHT
- removed net N$22: R22.1, SW2.RIGHT
- removed net N$33: R23.1, SW1.RIGHT
- new net N$15: R20.1, S4.1, S4.2, SW4.RIGHT
- new net N$17: R21.1, S3.1, S3.2, SW3.RIGHT
- new net N$24: R23.1, S1.1, S1.2, SW1.RIGHT
- new net N$4: IC1.21, R38.1
- new net N$5: R22.1, S2.1, S2.2, SW2.RIGHT
- net 1HZ: no longer R38.1
- net EXP1_32KHZ: now also IC2.5; no longer IC2.9
- net N$19: now also S5.1, S5.2
- net SW1: now also S1.3, S1.4
- net SW2: now also S2.3, S2.4
- net SW3: now also S3.3, S3.4
- net SW4: now also S4.3, S4.4
- net SW5: now also S5.3, S5.4
- net TCK: now also IC2.16
- net TDI: now also IC2.9
Routing:
- net +3V3: track 525.0 -> 558.8 mm, vias 8 -> 12
- net SW3: track 169.8 -> 189.7 mm, vias 0 -> 2
- net SW5: track 180.6 -> 162.2 mm, vias 0 -> 2
- net SW1: track 167.4 -> 156.1 mm, vias 0 -> 1
- net N$5: track 0.00 -> 11.1 mm
- net N$24: track 0.00 -> 10.6 mm
- net N$17: track 0.00 -> 10.5 mm
- net TCK: track 44.6 -> 54.6 mm
- net N$15: track 0.00 -> 9.81 mm
- net EXP1_32KHZ: track 157.5 -> 166.8 mm
- net SW4: track 179.4 -> 186.6 mm, vias 0 -> 1
- net SW2: track 169.5 -> 176.2 mm, vias 0 -> 1
- net N$19: track 3.40 -> 10.0 mm
- net N$21: track 4.19 -> 0.00 mm
- net N$22: track 3.93 -> 0.00 mm
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Other:
- board text added: "Copyright Colin O'Flynn 2012-2018"
- board text added: "TCK"
- board text added: "TDI"
- board text added: "TDO"
- board text added: "TMS"
- board text added: "rev04"
- board text removed: "Copyright Colin O'Flynn 2012"
- board text removed: "rev03"

Commit message: Fix bad pin numbering (closes #1) other minor additions
Parts:
- added U$2: (no value), oshw:OSHW_8MM
Routing:
- net N$4: track 0.00 -> 19.8 mm, vias 0 -> 2
Other:
- board text added: "50KHz/P12"
- board text added: "LED1/P1"
- board text added: "LED2/P2"
- board text added: "LED3/P3"
- board text added: "LED4/P4"
- board text added: "LED5/P5"
- board text added: "LED6/P6"
- board text added: "LED7/P7"
- board text added: "LED8/P8"
- board text added: "P26"
- board text added: "P27"
- board text added: "P28"
- board text added: "P29"
- board text added: "P30"
- board text added: "P33"
- board text added: "P34"
- board text removed: "32kHz/B1.10"
- board text removed: "B1.25"
- board text removed: "B1.26"
- board text removed: "B1.27"
- board text removed: "B1.28"
- board text removed: "B1.29"
- board text removed: "B1.32"
- board text removed: "B1.33"
- board text removed: "LED1/B2.100"
- board text removed: "LED2/B1.0"
- board text removed: "LED3/B1.1"
- board text removed: "LED4/B1.2"
- board text removed: "LED5/B1.3"
- board text removed: "LED6/B1.4"
- board text removed: "LED7/B1.5"
- board text removed: "LED8/B1.6"

Commit message: Fix net name for 32khz-->50khz, update schematic print
Connections:
- net EXP1_32KHZ renamed EXP1_50KHZ
Changed lines of the file:
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@@
 <wire x1="114.348" y1="82.25" x2="114.3" y2="82.298" width="0.254" layer="16"/>
 </signal>
-<signal name="EXP1_32KHZ">
+<signal name="EXP1_50KHZ">
 <contactref element="JP8" pad="1"/>
 <contactref element="JP12" pad="20"/>

Commit message: Small fixes to schematic
Parts:
- LED1, LED11, LED5: value (none) -> RED
- LED10, LED3, LED4, LED7, LED8, LED9: value (none) -> GRN
- LED2, LED6: value (none) -> YLW
- R10, R15, R6, R7, R8, R9: value (none) -> DNM
- R11: value (none) -> 330R
- R30: value (none) -> 51R
Changed lines of the file:
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@@
 <attribute name="OC_NEWARK" value="unknown" x="16.51" y="85.09" size="2.54" layer="27" font="vector" ratio="16" display="off"/>
 </element>
-<element name="LED1" library="led" package="CHIP-LED0805" value="" x="107.315" y="58.42" smashed="yes" rot="R270">
+<element name="LED1" library="led" package="CHIP-LED0805" value="RED" x="107.315" y="58.42" smashed="yes" rot="R270">
 <attribute name="VALUE" x="106.045" y="55.88" size="1.27" layer="27"/>
 </element>
-<element name="LED2" library="led" package="CHIP-LED0805" value="" x="107.315" y="55.88" smashed="yes" rot="R270">
+<element name="LED2" library="led" package="CHIP-LED0805" value="YLW" x="107.315" y="55.88" smashed="yes" rot="R270">
 <attribute name="VALUE" x="106.045" y="53.34" size="1.27" layer="27"/>
 </element>
-<element name="LED3" library="led" package="CHIP-LED0805" value="" x="107.315" y="53.34" smashed="yes" rot="R270">
+<element name="LED3" library="led" package="CHIP-LED0805" value="GRN" x="107.315" y="53.34" smashed="yes" rot="R270">
 <attribute name="VALUE" x="106.045" y="50.8" size="1.27" layer="27"/>
 </element>
-<element name="LED4" library="led" package="CHIP-LED0805" value="" x="107.315" y="50.8" smashed="yes" rot="R270">
+<element name="LED4" library="led" package="CHIP-LED0805" value="GRN" x="107.315" y="50.8" smashed="yes" rot="R270">
 <attribute name="VALUE" x="106.045" y="48.26" size="1.27" layer="27"/>
 </element>
-<element name="LED5" library="led" package="CHIP-LED0805" value="" x="107.315" y="48.26" smashed="yes" rot="R270">
+<element name="LED5" library="led" package="CHIP-LED0805" value="RED" x="107.315" y="48.26" smashed="yes" rot="R270">
 <attribute name="VALUE" x="106.045" y="45.72" size="1.27" layer="27"/>
 </element>
-<element name="LED6" library="led" package="CHIP-LED0805" value="" x="107.315" y="45.72" smashed="yes" rot="R270">
+<element name="LED6" library="led" package="CHIP-LED0805" value="YLW" x="107.315" y="45.72" smashed="yes" rot="R270">
 <attribute name="VALUE" x="106.045" y="43.18" size="1.27" layer="27"/>
 </element>
-<element name="LED7" library="led" package="CHIP-LED0805" value="" x="107.315" y="43.18" smashed="yes" rot="R270">
+<element name="LED7" library="led" package="CHIP-LED0805" value="GRN" x="107.315" y="43.18" smashed="yes" rot="R270">
 <attribute name="VALUE" x="106.045" y="40.64" size="1.27" layer="27"/>
 </element>
-<element name="LED8" library="led" package="CHIP-LED0805" value="" x="107.315" y="40.64" smashed="yes" rot="R270">
+<element name="LED8" library="led" package="CHIP-LED0805" value="GRN" x="107.315" y="40.64" smashed="yes" rot="R270">
 <attribute name="VALUE" x="106.045" y="38.1" size="1.27" layer="27"/>
 </element>
@@
 <element name="SW4" library="customs" package="SS-12E10" value="SS-12E10" x="10.16" y="22.86" smashed="yes"/>
 <element name="SW5" library="customs" package="SS-12E10" value="SS-12E10" x="10.16" y="13.97" smashed="yes"/>
-<element name="R6" library="resistor" package="R0603" value="" x="40.259" y="42.037" smashed="yes" rot="MR180">
+<element name="R6" library="resistor" package="R0603" value="DNM" x="40.259" y="42.037" smashed="yes" rot="MR180">
 <attribute name="NAME" x="41.87" y="42.648" size="1.27" layer="26" font="vector" ratio="15" rot="MR180"/>
 <attribute name="VALUE" x="39.37" y="44.069" size="1.27" layer="28" rot="MR180"/>
 </element>
-<element name="R7" library="resistor" package="R0603" value="" x="40.259" y="39.37" smashed="yes" rot="MR180">
+<element name="R7" library="resistor" package="R0603" value="DNM" x="40.259" y="39.37" smashed="yes" rot="MR180">
 <attribute name="NAME" x="41.87" y="39.981" size="1.27" layer="26" font="vector" ratio="15" rot="MR180"/>
 <attribute name="VALUE" x="39.37" y="41.402" size="1.27" layer="28" rot="MR180"/>
 </element>
-<element name="R8" library="resistor" package="R0603" value="" x="40.259" y="36.83" smashed="yes" rot="MR180">
+<element name="R8" library="resistor" package="R0603" value="DNM" x="40.259" y="36.83" smashed="yes" rot="MR180">
 <attribute name="NAME" x="41.87" y="37.441" size="1.27" layer="26" font="vector" ratio="15" rot="MR180"/>
 <attribute name="VALUE" x="39.37" y="38.862" size="1.27" layer="28" rot="MR180"/>
 </element>
-<element name="R9" library="resistor" package="R0603" value="" x="40.259" y="34.29" smashed="yes" rot="MR180">
+<element name="R9" library="resistor" package="R0603" value="DNM" x="40.259" y="34.29" smashed="yes" rot="MR180">
 <attribute name="NAME" x="41.87" y="34.901" size="1.27" layer="26" font="vector" ratio="15" rot="MR180"/>
 <attribute name="VALUE" x="39.37" y="36.322" size="1.27" layer="28" rot="MR180"/>
 </element>
-<element name="R10" library="resistor" package="R0603" value="" x="19.05" y="11.176" smashed="yes" rot="MR180">
+<element name="R10" library="resistor" package="R0603" value="DNM" x="19.05" y="11.176" smashed="yes" rot="MR180">
 <attribute name="NAME" x="21.161" y="11.787" size="1.27" layer="26" font="vector" ratio="15" rot="MR180"/>
 <attribute name="VALUE" x="18.161" y="13.208" size="1.27" layer="28" rot="MR180"/>
@@
 </element>
 <element name="SW6" library="customs" package="SS-12E10" value="SS-12E10" x="119.126" y="23.622" smashed="yes" rot="R270"/>
-<element name="R15" library="resistor" package="R0603" value="" x="120.05" y="34.3" smashed="yes" rot="MR180">
+<element name="R15" library="resistor" package="R0603" value="DNM" x="120.05" y="34.3" smashed="yes" rot="MR180">
 <attribute name="NAME" x="114.62" y="35.031" size="1.27" layer="26" font="vector" ratio="15" rot="MR180"/>
 <attribute name="VALUE" x="119.161" y="36.332" size="1.27" layer="28" rot="MR180"/>
@@
 <attribute name="VALUE" x="105.197" y="81.597" size="1.27" layer="28" font="vector" ratio="15" rot="MR180"/>
 </element>
-<element name="LED9" library="led" package="CHIP-LED0805" value="" x="115.316" y="87.884" smashed="yes" rot="R270">
+<element name="LED9" library="led" package="CHIP-LED0805" value="GRN" x="115.316" y="87.884" smashed="yes" rot="R270">
 <attribute name="VALUE" x="114.046" y="85.344" size="1.27" layer="27"/>
 </element>
@@
 <attribute name="VALUE" x="108.645" y="93.455" size="1.27" layer="28" font="vector" ratio="15" rot="MR180"/>
 </element>
-<element name="LED10" library="led" package="CHIP-LED0805" value="" x="115.316" y="91.186" smashed="yes" rot="R270">
+<element name="LED10" library="led" package="CHIP-LED0805" value="GRN" x="115.316" y="91.186" smashed="yes" rot="R270">
 <attribute name="VALUE" x="114.046" y="88.646" size="1.27" layer="27"/>
 </element>
@@
 <attribute name="VALUE" x="110.115" y="61.2599" size="1.27" layer="28" font="vector" ratio="15" rot="MR0"/>
 </element>
-<element name="R30" library="rcl" package="R0603" value="" x="97.247" y="65.695" smashed="yes" rot="MR0">
+<element name="R30" library="rcl" package="R0603" value="51R" x="97.247" y="65.695" smashed="yes" rot="MR0">
 <attribute name="NAME" x="98.582" y="66.68" size="1.27" layer="26" font="vector" ratio="15" rot="MR0"/>
 <attribute name="VALUE" x="97.882" y="63.79" size="1.27" layer="28" rot="MR0"/>
@@
 <attribute name="VALUE" x="96.464" y="49.212" size="1.27" layer="28" font="vector" ratio="15" rot="MR180"/>
 </element>
-<element name="R11" library="resistor" package="R0603" value="" x="97.353" y="44.625" smashed="yes" rot="MR180">
+<element name="R11" library="resistor" package="R0603" value="330R" x="97.353" y="44.625" smashed="yes" rot="MR180">
 <attribute name="NAME" x="99.264" y="45.136" size="1.27" layer="26" font="vector" ratio="15" rot="MR180"/>
 <attribute name="VALUE" x="96.464" y="46.657" size="1.27" layer="28" rot="MR180"/>
@@
 <attribute name="VALUE" x="112.285" y="92.595" size="1.27" layer="28" font="vector" ratio="15" rot="MR0"/>
 </element>
-<element name="LED11" library="led" package="CHIP-LED0805" value="" x="75.7428" y="34.29" smashed="yes" rot="MR90">
+<element name="LED11" library="led" package="CHIP-LED0805" value="RED" x="75.7428" y="34.29" smashed="yes" rot="MR90">
 <attribute name="VALUE" x="74.4728" y="36.83" size="1.27" layer="28" rot="MR180"/>
 </element>
